Commit message: Adding missing packages; ur5_smartlab and ur5_smarlab_gazebo

File: ur5_smartlab/urdf/ur5_smartlab.xacro (robot description, xacro)
@@ -6,37 +6,42 @@
     <xacro:include filename="$(find ur_description)/urdf/ur5.urdf.xacro"/>
     <!-- arm -->
-    <xacro:ur5_robot prefix="" joint_limited="false"/>
+    <!--<xacro:ur5_robot prefix="" joint_limited="false"/>-->
     <!-- arm -->
-    <!--<xacro:ur5_robot prefix="" joint_limited="true"-->
-                     <!--shoulder_pan_lower_limit="${-pi}" shoulder_pan_upper_limit="${pi}"-->
-                     <!--shoulder_lift_lower_limit="${-pi}" shoulder_lift_upper_limit="${pi}"-->
-                     <!--elbow_joint_lower_limit="${-pi}" elbow_joint_upper_limit="${pi}"-->
-                     <!--wrist_1_lower_limit="${-pi}" wrist_1_upper_limit="${pi}"-->
-                     <!--wrist_2_lower_limit="${-pi}" wrist_2_upper_limit="${pi}"-->
-                     <!--wrist_3_lower_limit="${-pi}" wrist_3_upper_limit="${pi}"/>-->
+    <xacro:ur5_robot prefix="" joint_limited="true"
+                     shoulder_pan_lower_limit="${-pi}" shoulder_pan_upper_limit="${pi}"
+                     shoulder_lift_lower_limit="${-pi}" shoulder_lift_upper_limit="${pi}"
+                     elbow_joint_lower_limit="${-pi}" elbow_joint_upper_limit="${pi}"
+                     wrist_1_lower_limit="${-pi}" wrist_1_upper_limit="${pi}"
+                     wrist_2_lower_limit="${-pi}" wrist_2_upper_limit="${pi}"
+                     wrist_3_lower_limit="${-pi}" wrist_3_upper_limit="${pi}"/>
     <xacro:include filename="$(find ur5_smartlab)/urdf/world.xacro"/>
     <material name="DarkPlastic">
         <color rgba="0.1 0.1 0.1 1"/>
     </material>
-    <!--<link name="gelsight">-->
-        <!--<visual>-->
-            <!--<origin xyz="0.035 0 0" rpy="0 ${-pi/2} 0"/>-->
-            <!--<geometry>-->
-                <!--<cylinder radius="0.03" length="0.07"/>-->
-            <!--</geometry>-->
-            <!--<material name="DarkPlastic"/>-->
-        <!--</visual>-->
-        <!--<collision>-->
-            <!--<origin xyz="0.035 0 0" rpy="0 ${-pi/2} 0"/>-->
-            <!--<geometry>-->
-                <!--<cylinder radius="0.03" length="0.07"/>-->
-            <!--</geometry>-->
-        <!--</collision>-->
-    <!--</link>-->
-    <!--<joint name="robot_to_gelsight" type="fixed">-->
-        <!--<parent link="ee_link"/>-->
-        <!--<child link="gelsight"/>-->
-        <!--<origin xyz="0.0 0.0 0.0" rpy="0.0 0.0 0.0"/>-->
-    <!--</joint>-->
+    <link name="gelsight">
+        <!--<inertial>-->
+            <!--<origin xyz="0 0 0.5" rpy="0 0 0"/>-->
+            <!--<mass value="0"/>-->
+            <!--<inertia ixx="100" ixy="0" ixz="0" iyy="100" iyz="0" izz="100"/>-->
+        <!--</inertial>-->
+        <visual>
+            <origin xyz="0.035 0 0" rpy="0 ${-pi/2} 0"/>
+            <geometry>
+                <cylinder radius="0.03" length="0.07"/>
+            </geometry>
+            <material name="DarkPlastic"/>
+        </visual>
+        <collision>
+            <origin xyz="0.035 0 0" rpy="0 ${-pi/2} 0"/>
+            <geometry>
+                <cylinder radius="0.03" length="0.07"/>
+            </geometry>
+        </collision>
+    </link>
+    <joint name="robot_to_gelsight" type="fixed">
+        <parent link="ee_link"/>
+        <child link="gelsight"/>
+        <origin xyz="0.0 0.0 0.0" rpy="0.0 0.0 0.0"/>
+    </joint>
     <joint name="table_to_robot" type="fixed">
         <parent link="table"/>
